File: ver2.0 + design/ver3.0+VinSeparat.brd (EAGLE design)
At the start: 160.1 x 99.5 mm, 65 parts

Commit message: corectare trasee
Parts:
- moved C2 42.2 mm to (177.2, 20.1)
- moved C3 42.2 mm to (177.2, 24.6)
- moved C4 42.2 mm to (177.2, 30.4)
- moved C5 42.2 mm to (177.2, 37.1)
- moved C6 42.2 mm to (177.2, 43.7)
- moved C7 42.2 mm to (176.8, 51.9)
- moved C8 42.2 mm to (176.8, 63.9)
- moved C12 22.0 mm to (-6.44, 37.6)
- moved C13 22.0 mm to (-6.09, 42.6)
- moved C14 22.0 mm to (-6.74, 48.6)
- moved C15 22.0 mm to (-6.39, 53.6)
- moved C16 22.0 mm to (-6.04, 58.6)
- moved C17 22.0 mm to (-6.69, 68.6)
- moved C_SS 3.00 mm to (82.9, 14.3)
Routing:
- net VCC: track 28.0 -> 24.3 mm, vias 1 -> 0
- net GND: track 78.4 -> 81.7 mm
- net N$11: track 8.05 -> 11.0 mm
- net SW: track 75.1 -> 76.8 mm
- net N$3: track 33.7 -> 34.4 mm
- net VOUT: track 20.3 -> 20.9 mm
