File: lm3150/ver1.brd (EAGLE design)
At the start: 160 x 100 mm, 24 parts, among them P1 BANANA, P2 BANANA, P3 BANANA, P4 BANANA, P5 BANANA

Commit message: 04.04.2018
Parts:
- added KK3, KK4: SK95-2M3, heatsink:SK95-2M3
- moved U$3 117.3 mm to (77.5, 50.8)
- moved U$2 108.7 mm to (77.5, 43.2)
- moved U$5 67.9 mm to (82.5, 7.62), turned to 0 degrees
- moved U$4 64.8 mm to (82.5, 18.1), turned to 0 degrees
- moved CVCC 39.2 mm to (28.9, 28.6)
- moved P1 39.2 mm to (8.89, 50.8)
- moved Q2_LOW 39.2 mm to (41.3, 40.6)
- moved RFB2.2 39.2 mm to (19.1, 25.1)
- moved CBST 39.2 mm to (35.6, 17.8)
- moved CBYP 39.2 mm to (30.2, 18.1)
- moved CEN 39.2 mm to (32.1, 28.6)
- moved CFF 39.2 mm to (24.1, 16.8)
- moved CSS 39.2 mm to (35.2, 28.6)
- moved L2 39.2 mm to (50.8, 34.3)
- moved P3 39.2 mm to (58.4, 26.0)
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Routing:
- net N$9: track 0.00 -> 116.8 mm
- net N$8: track 0.00 -> 86.4 mm
Other:
- board size 160 x 100 mm -> 66 x 58.1 mm
- board text added: "External Capacitors"
- board text added: "Reserve Mossfet"
