File: lm3150/ver1.sch (EAGLE design)
At the start: 24 parts, among them P1 BANANA, P2 BANANA, P3 BANANA, P4 BANANA, P5 BANANA

Commit message: 04.04.2018
Parts:
- added KK3, KK4: SK95-2M3, heatsink:SK95-2M3
Changed lines of the file:
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@@
 <setting verticaltext="up"/>
 </settings>
-<grid distance="0.05" unitdist="inch" unit="inch" style="lines" multiple="1" display="yes" altdistance="0.0125" altunitdist="inch" altunit="inch"/>
+<grid distance="0.1" unitdist="inch" unit="inch" style="lines" multiple="1" display="no" altdistance="0.01" altunitdist="inch" altunit="inch"/>
 <layers>
 <layer number="1" name="Top" color="4" fill="1" visible="yes" active="no"/>
@@
 <layer number="56" name="wert" color="7" fill="1" visible="yes" active="no"/>
 <layer number="57" name="tCAD" color="7" fill="1" visible="yes" active="no"/>
-<layer number="59" name="tCarbon" color="7" fill="1" visible="no" active="no"/>
-<layer number="60" name="bCarbon" color="7" fill="1" visible="no" active="no"/>
+<layer number="59" name="tCarbon" color="7" fill="1" visible="yes" active="no"/>
+<layer number="60" name="bCarbon" color="7" fill="1" visible="yes" active="no"/>
 <layer number="90" name="Modules" color="5" fill="1" visible="yes" active="yes"/>
 <layer number="91" name="Nets" color="2" fill="1" visible="yes" active="yes"/>
@@
 <part name="U$5" library="H_bridge_library" deviceset="BANANA" device=""/>
 <part name="P5" library="adi_v1.6" deviceset="BANANA" device=""/>
+<part name="KK3" library="heatsink" deviceset="SK95-2M3" device=""/>
+<part name="KK4" library="heatsink" deviceset="SK95-2M3" device=""/>
 </parts>
 <sheets>
@@
 <instance part="U$5" gate="G$1" x="72.39" y="-14.2875"/>
 <instance part="P5" gate="G$1" x="64.77" y="-13.6525" rot="R180"/>
+<instance part="KK3" gate="G$1" x="96.52" y="15.24" rot="R270"/>
+<instance part="KK4" gate="G$1" x="106.68" y="15.24" rot="R270"/>
 </instances>
 <busses>
